File: P.003-V1.0.1/P.003-V1.0.1.kicad_pcb (KiCad board)
At the start: 2 copper layers, 19 parts, among them Q1 BS250, SW1 ON/OFF, SW2 Mode, SW3 Roll, U1 ATtiny85-20P, U2 74HC595

Commit message: add 3d and footprint
Parts:
- SW1: footprint Button_Switch_THT:SW_Slide-03_Wuerth-WS-SLTV_10x2.5x6.4_P2.54mm -> Button_Switch_THT:SW_Slide_SPDT_Straight_CK_OS102011MS2Q
Connections:
- SW1 pad 2: unconnected-(SW1-C-Pad2) -> Net-(Q1-D)
- SW1 pad 3: Net-(Q1-D) -> unconnected-(SW1-A-Pad3)

Commit message: Review OK
Parts:
- moved R10 64.6 mm to (125.6, 132.9), turned to 0 degrees
- moved U2 60.9 mm to (166.2, 67.0)
- moved R9 59.9 mm to (125.6, 128.8), turned to 0 degrees
- moved R8 55.5 mm to (125.6, 124.8), turned to 0 degrees
- moved R7 51.3 mm to (125.6, 120.7), turned to 0 degrees
- moved SW2 50.8 mm to (162.0, 107.8)
- moved R6 47.5 mm to (125.6, 116.7), turned to 0 degrees
- moved SW1 46.2 mm to (141.3, 95.9)
- moved R5 44.0 mm to (125.6, 112.6), turned to 0 degrees
- moved R4 41.1 mm to (125.6, 108.6), turned to 0 degrees
- moved R3 38.8 mm to (125.6, 104.5), turned to 0 degrees
- moved R2 36.8 mm to (125.6, 98.5), turned to 0 degrees
- moved R1 36.5 mm to (125.6, 94.4), turned to 0 degrees
- moved U1 35.2 mm to (178.2, 104.5)
- moved Q1 31.6 mm to (151.2, 95.7)
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
Commit message: first try
Parts:
- SW2, SW3: footprint Button_Switch_THT:SW_PUSH-12mm -> Button_Switch_THT:SW_PUSH_6mm_H4.3mm
- moved R3 93.1 mm to (207.0, 59.4), turned to -90 degrees
- moved R4 90.9 mm to (202.0, 59.4), turned to -90 degrees
- moved R5 89.1 mm to (197.0, 59.4), turned to -90 degrees
- moved R6 87.7 mm to (192.0, 59.4), turned to -90 degrees
- moved R2 86.6 mm to (209.1, 75.5), turned to 180 degrees
- moved R7 79.6 mm to (187.0, 70.1), turned to 90 degrees
- moved R8 78.6 mm to (182.0, 70.0), turned to 90 degrees
- moved R9 78.5 mm to (177.0, 69.6), turned to 90 degrees
- moved R10 78.2 mm to (171.5, 69.6), turned to 90 degrees
- moved Q1 77.3 mm to (205.0, 40.0)
- moved BT1 67.4 mm to (190.0, 30.5), turned to 180 degrees
- moved D1 58.7 mm to (172.7, 38.5)
- moved R1 57.4 mm to (179.6, 75.0), turned to 180 degrees
- moved U1 57.1 mm to (177.2, 47.4)
- moved SW3 56.8 mm to (200.8, 81.8)
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
Commit message: Posicao
Parts:
- moved R3 82.9 mm to (136.1, 102.3), turned to 90 degrees
- moved R4 77.9 mm to (131.3, 92.2)
- moved R5 77.6 mm to (126.6, 92.2)
- moved R6 77.4 mm to (121.8, 92.2)
- moved R7 77.0 mm to (117.1, 102.3)
- moved R8 76.8 mm to (112.3, 102.3)
- moved R2 73.3 mm to (140.8, 102.3), turned to 90 degrees
- moved SW3 71.6 mm to (139.0, 118.0)
- moved Q1 70.7 mm to (143.0, 74.1)
- moved D1 69.8 mm to (112.5, 73.8)
- moved SW2 69.4 mm to (112.5, 118.0)
- moved U2 68.7 mm to (146.4, 80.2)
- moved BT1 68.4 mm to (129.0, 61.5)
- moved AFF1 68.4 mm to (123.9, 122.5)
- moved U1 68.4 mm to (117.2, 80.2)
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
Commit message: add
Parts:
- added ?: MountingHole_3.2mm_M3, MountingHole:MountingHole_3.2mm_M3, F.Cu at (112.0, 52.0)
- added ?: MountingHole_3.2mm_M3, MountingHole:MountingHole_3.2mm_M3, F.Cu at (146.0, 52.0)
- moved SW2 1.27 mm to (112.2, 116.7)
- moved SW3 1.27 mm to (139.2, 116.7)
- moved R10 0.25 mm to (120.6, 107.2)
- moved R9 0.25 mm to (137.4, 107.2)
Routing:
- net /Attiny85/VIN+: track 0.00 -> 93.8 mm
- net Net-(BT1-+): track 0.00 -> 70.2 mm
- net Net-(D1-A): track 0.00 -> 59.3 mm
- net Net-(U1-XTAL2/PB4): track 0.00 -> 58.9 mm
- net Net-(Q1-G): track 0.00 -> 51.8 mm
- net Net-(U1-XTAL1/PB3): track 0.00 -> 44.9 mm
- net /Display 7 Segment/Q7: track 0.00 -> 44.6 mm
- net Net-(Q1-D): track 0.00 -> 43.6 mm
- net /Display 7 Segment/Q4: track 0.00 -> 39.4 mm
- net /Display 7 Segment/Q6: track 0.00 -> 38.6 mm
- net /Display 7 Segment/Q5: track 0.00 -> 36.8 mm
- net Net-(AFF1-c): track 0.00 -> 34.4 mm
- net /Display 7 Segment/Q2: track 0.00 -> 28.0 mm
- net /Display 7 Segment/Q3: track 0.00 -> 27.5 mm
- net /Display 7 Segment/Q1: track 0.00 -> 27.3 mm
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- added copper zone on B.Cu, net /Attiny85/VIN-
- added copper zone on F.Cu, net /Attiny85/VIN-
Other:
- board outline added: 42 x 78.5 mm
- board text added: "GSAS - LABS P. 003 V. 1.0.1"
- board text added: "Mode/Select"
- board text added: "Roll/Reset"
