File: P.003-V1.0.1/P.003-V1.0.1.kicad_pcb (KiCad board)
At the start: 2 copper layers, 42 x 78.5 mm, 21 parts, among them Q1 BS250, SW1 ON/OFF, SW2 Mode, SW3 Roll, U1 ATtiny85-20P, U2 74HC595

Commit message: update values
Parts:
- R10, R3, R4, R5, R6, R7, R8, R9: value 470 -> 1K
- R2: value 1K -> 2.2K
Changed lines of the file:
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@@
 			)
 		)
-		(property "Value" "470"
+		(property "Value" "1K"
 			(at 5.08 2.37 90)
 			(layer "F.Fab")
@@
 			)
 		)
-		(property "Value" "470"
+		(property "Value" "1K"
 			(at 5.08 2.37 90)
 			(layer "F.Fab")
@@
 			)
 		)
-		(property "Value" "470"
+		(property "Value" "1K"
 			(at 5.08 2.37 90)
 			(layer "F.Fab")
@@
 			)
 		)
-		(property "Value" "470"
+		(property "Value" "1K"
 			(at 5.08 2.37 90)
 			(layer "F.Fab")
@@
 			)
 		)
-		(property "Value" "470"
+		(property "Value" "1K"
 			(at 5.08 2.37 0)
 			(layer "F.Fab")
@@
 			)
 		)
-		(property "Value" "1K"
+		(property "Value" "2.2K"
 			(at 5.08 2.37 90)
 			(layer "F.Fab")
@@
 			)
 		)
-		(property "Value" "470"
+		(property "Value" "1K"
 			(at 5.08 2.37 90)
 			(layer "F.Fab")
@@
 			)
 		)
-		(property "Value" "470"
+		(property "Value" "1K"
 			(at 5.08 2.37 0)
 			(layer "F.Fab")
@@
 			)
 		)
-		(property "Value" "470"
+		(property "Value" "1K"
 			(at 5.08 2.37 90)
 			(layer "F.Fab")
