File: P.003-V1.0.1/7_segment_display.kicad_sch (KiCad schematic)
At the start: 0 parts

Commit message: add kicad
Parts:
- added AFF1: LTS-6980HR, Display_7Segment:7SegmentLED_LTS6760_LTS6780, symbol Display_Character:LTS-6980HR
- added R10, R3, R4, R5, R6, R7, R8, R9: R, symbol Device:R

Commit message: Schematic wired
Parts:
- AFF1: value LTS-6980HR -> Display
- R10, R3, R4, R5, R6, R7, R8, R9: value R -> 470
Connections:
- net at AFF1.1 (e): now also R7.1
- net at AFF1.10 (g): now also R9.1
- net at AFF1.2 (d): now also R6.2
- net VIN-: now reaches AFF1.3 (C.K.)
- net VIN-: now also AFF1.8 (C.K.)
- net at AFF1.4 (c): now also R5.2
- net at AFF1.5 (DP): now also R10.1
- net at AFF1.6 (b): now also R4.2
- net at AFF1.7 (a): now also R3.1
- net at AFF1.9 (f): now also R8.1
- net Q3: now reaches R6.1
- net Q2: now reaches R5.1
- net Q0: now reaches R3.2
- net Q5: now reaches R8.2
- net Q4: now reaches R7.2
- net Q6: now reaches R9.2
- net Q1: now reaches R4.1
- net Q7: now reaches R10.2
Other:
- company: (none) -> GSAS - Labs
- title: (none) -> Display 7 Segment
- moved on the sheet: AFF1

Commit message: add footprint
Parts:
- R10, R3, R4, R5, R6, R7, R8, R9: footprint (none) -> Resistor_THT:R_Axial_DIN0207_L6.3mm_D2.5mm_P10.16mm_Horizontal
Changed lines of the file:
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@@
 			)
 		)
-		(property "Footprint" ""
+		(property "Footprint" "Resistor_THT:R_Axial_DIN0207_L6.3mm_D2.5mm_P10.16mm_Horizontal"
 			(at 121.92 126.492 90)
 			(hide yes)
@@
 			)
 		)
-		(property "Footprint" ""
+		(property "Footprint" "Resistor_THT:R_Axial_DIN0207_L6.3mm_D2.5mm_P10.16mm_Horizontal"
 			(at 121.92 96.012 90)
 			(hide yes)
@@
 			)
 		)
-		(property "Footprint" ""
+		(property "Footprint" "Resistor_THT:R_Axial_DIN0207_L6.3mm_D2.5mm_P10.16mm_Horizontal"
 			(at 121.92 69.088 90)
 			(hide yes)
@@
 			)
 		)
-		(property "Footprint" ""
+		(property "Footprint" "Resistor_THT:R_Axial_DIN0207_L6.3mm_D2.5mm_P10.16mm_Horizontal"
 			(at 121.92 89.408 90)
 			(hide yes)
@@
 			)
 		)
-		(property "Footprint" ""
+		(property "Footprint" "Resistor_THT:R_Axial_DIN0207_L6.3mm_D2.5mm_P10.16mm_Horizontal"
 			(at 121.92 55.372 90)
 			(hide yes)
@@
 			)
 		)
-		(property "Footprint" ""
+		(property "Footprint" "Resistor_THT:R_Axial_DIN0207_L6.3mm_D2.5mm_P10.16mm_Horizontal"
 			(at 121.92 106.172 90)
 			(hide yes)
@@
 			)
 		)
-		(property "Footprint" ""
+		(property "Footprint" "Resistor_THT:R_Axial_DIN0207_L6.3mm_D2.5mm_P10.16mm_Horizontal"
 			(at 121.92 79.248 90)
 			(hide yes)
@@
 			)
 		)
-		(property "Footprint" ""
+		(property "Footprint" "Resistor_THT:R_Axial_DIN0207_L6.3mm_D2.5mm_P10.16mm_Horizontal"
 			(at 121.92 116.332 90)
 			(hide yes)

Commit message: update values
Parts:
- R10, R3, R4, R5, R6, R7, R8, R9: value 470 -> 1K
Changed lines of the file:
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@@
 	(title_block
 		(title "Display 7 Segment")
-		(date "2026-08-23")
+		(date "2026-09-13")
 		(rev "01")
 		(company "GSAS - Labs")
@@
 			)
 		)
-		(property "Value" "470"
+		(property "Value" "1K"
 			(at 121.92 124.46 90)
 			(show_name no)
@@
 			)
 		)
-		(property "Value" "470"
+		(property "Value" "1K"
 			(at 121.92 93.98 90)
 			(show_name no)
@@
 			)
 		)
-		(property "Value" "470"
+		(property "Value" "1K"
 			(at 121.92 63.5 90)
 			(show_name no)
@@
 			)
 		)
-		(property "Value" "470"
+		(property "Value" "1K"
 			(at 121.92 83.82 90)
 			(show_name no)
@@
 			)
 		)
-		(property "Value" "470"
+		(property "Value" "1K"
 			(at 121.92 53.34 90)
 			(show_name no)
@@
 			)
 		)
-		(property "Value" "470"
+		(property "Value" "1K"
 			(at 121.92 104.14 90)
 			(show_name no)
@@
 			)
 		)
-		(property "Value" "470"
+		(property "Value" "1K"
 			(at 121.92 73.66 90)
 			(show_name no)
@@
 			)
 		)
-		(property "Value" "470"
+		(property "Value" "1K"
 			(at 121.92 114.3 90)
 			(show_name no)
