File: P.003-V1.0.1/power_supply.kicad_sch (KiCad schematic)
At the start: 0 parts

Commit message: add kicad
Parts:
- added BT1: 3V, symbol Device:Battery_Cell
- added D1: LED, symbol Device:LED
- added Q1: BS250, Package_TO_SOT_THT:TO-92_Inline, symbol Transistor_FET:BS250
- added R1: 100K, symbol Device:R
- added R2: 1K, symbol Device:R
- added SW1: ON/OFF, Button_Switch_THT:SW_Slide-03_Wuerth-WS-SLTV_10x2.5x6.4_P2.54mm, symbol Switch:SW_Wuerth_450301014042
Connections:
- new net: BT1.1 (+), SW1.1 (B)
- new net: Q1.1 (D), SW1.3 (A)
- new net: Q1.2 (G), R1.1
- new net: D1.2 (A), R2.2
- new net VIN+: Q1.3 (S), R2.1
- new net VIN-: BT1.2 (-), D1.1 (K), R1.2
- no-connect marks 0 -> 1

Commit message: Schematic wired
Other:
- company: (none) -> GSAS - Labs
- title: (none) -> Power Supply
- moved on the sheet: BT1, D1, Q1, R1, R2, SW1

Commit message: add footprint
Parts:
- BT1: footprint (none) -> Battery:BatteryHolder_Keystone_3008_1x2450
- D1: footprint (none) -> LED_THT:LED_D3.0mm
- R1, R2: footprint (none) -> Resistor_THT:R_Axial_DIN0207_L6.3mm_D2.5mm_P10.16mm_Horizontal
Changed lines of the file:
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@@
 			)
 		)
-		(property "Footprint" ""
+		(property "Footprint" "Battery:BatteryHolder_Keystone_3008_1x2450"
 			(at 114.3 105.156 90)
 			(hide yes)
@@
 			)
 		)
-		(property "Footprint" ""
+		(property "Footprint" "Resistor_THT:R_Axial_DIN0207_L6.3mm_D2.5mm_P10.16mm_Horizontal"
 			(at 149.352 107.95 90)
 			(hide yes)
@@
 			)
 		)
-		(property "Footprint" ""
+		(property "Footprint" "LED_THT:LED_D3.0mm"
 			(at 162.56 110.49 0)
 			(hide yes)
@@
 			)
 		)
-		(property "Footprint" ""
+		(property "Footprint" "Resistor_THT:R_Axial_DIN0207_L6.3mm_D2.5mm_P10.16mm_Horizontal"
 			(at 160.782 100.33 90)
 			(hide yes)

Commit message: add 3d and footprint
Parts:
- SW1: footprint Button_Switch_THT:SW_Slide-03_Wuerth-WS-SLTV_10x2.5x6.4_P2.54mm -> Button_Switch_THT:SW_Slide_SPDT_Straight_CK_OS102011MS2Q
Connections:
- net at SW1.2 (C): now also Q1.1 (D)
- net at SW1.3 (A): no longer Q1.1 (D)
Changed lines of the file:
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@@
 	)
 	(no_connect
-		(at 135.89 97.79)
+		(at 135.89 92.71)
 	)
 	(wire
@@
 	(wire
 		(pts
+			(xy 142.24 97.79) (xy 142.24 92.71)
+		)
+		(stroke
+			(width 0)
+			(type default)
+		)
+	)
+	(wire
+		(pts
 			(xy 151.13 116.84) (xy 114.3 116.84)
 		)
@@
 	(wire
 		(pts
+			(xy 135.89 97.79) (xy 142.24 97.79)
+		)
+		(stroke
+			(width 0)
+			(type default)
+		)
+	)
+	(wire
+		(pts
 			(xy 162.56 92.71) (xy 162.56 96.52)
 		)
@@
 	(wire
 		(pts
+			(xy 142.24 92.71) (xy 146.05 92.71)
+		)
+		(stroke
+			(width 0)
+			(type default)
+		)
+	)
+	(wire
+		(pts
 			(xy 162.56 116.84) (xy 151.13 116.84)
-		)
-		(stroke
-			(width 0)
-			(type default)
-		)
-	)
-	(wire
-		(pts
-			(xy 135.89 92.71) (xy 146.05 92.71)
 		)
 		(stroke
@@
 			)
 		)
-		(property "Footprint" "Button_Switch_THT:SW_Slide-03_Wuerth-WS-SLTV_10x2.5x6.4_P2.54mm"
+		(property "Footprint" "Button_Switch_THT:SW_Slide_SPDT_Straight_CK_OS102011MS2Q"
 			(at 130.81 105.41 0)
 			(hide yes)

Commit message: update values
Parts:
- R2: value 1K -> 2.2K
Changed lines of the file:
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@@
 	(title_block
 		(title "Power Supply")
-		(date "2026-08-23")
+		(date "2026-09-13")
 		(rev "01")
 		(company "GSAS - Labs")
@@
 			)
 		)
-		(property "Value" "1K"
+		(property "Value" "2.2K"
 			(at 165.1 101.5999 0)
 			(show_name no)
