File: P.003-V1.0.1/shift_register_74HC595.kicad_sch (KiCad schematic)
At the start: 0 parts

Commit message: add kicad
Parts:
- added U2: 74HC595, symbol 74xx:74HC595
Changed lines of the file:
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@@
 	(generator_version "10.0")
 	(paper "A4")
+	(hierarchical_label "VIN+"
+		(shape input)
+		(at 116.84 73.66 180)
+		(effects
+			(font
+				(size 1.27 1.27)
+			)
+			(justify right)
+		)
+	)
+	(hierarchical_label "VIN-"
+		(shape input)
+		(at 116.84 80.01 180)
+		(effects
+			(font
+				(size 1.27 1.27)
+			)
+			(justify right)
+		)
+	)
+	(symbol
+		(lib_id "74xx:74HC595")
+		(at 137.16 93.98 0)
+		(unit 1)
+		(body_style 1)
+		(exclude_from_sim no)
+		(in_bom yes)
+		(on_board yes)
+		(in_pos_files yes)
+		(dnp no)
+		(fields_autoplaced yes)
+		(property "Reference" "U2"
+			(at 139.3033 76.2 0)
+			(show_name no)
+			(do_not_autoplace no)
+			(effects
+				(font
+					(size 1.27 1.27)
+				)
+				(justify left)
+			)
+		)
+		(property "Value" "74HC595"
+			(at 139.3033 78.74 0)
+			(show_name no)
+			(do_not_autoplace no)
+			(effects
+				(font
+					(size 1.27 1.27)
+				)
+				(justify left)
+			)
+		)
+		(property "Footprint" ""
+			(at 137.16 93.98 0)
+			(hide yes)
+			(show_name no)
+			(do_not_autoplace no)
+			(effects
+				(font
+					(size 1.27 1.27)
+				)
+			)
+		)
+		(property "Datasheet" "http://www.ti.com/lit/ds/symlink/sn74hc595.pdf"
+			(at 137.16 93.98 0)
+			(hide yes)
+			(show_name no)
+			(do_not_autoplace no)
+			(effects
+				(font
+					(size 1.27 1.27)
+				)
+			)
+		)
+		(property "Description" "8-bit serial in/out Shift Register 3-State Outputs"
+			(at 137.16 93.98 0)
+			(hide yes)
+			(show_name no)
+			(do_not_autoplace no)
+			(effects
+				(font
+					(size 1.27 1.27)
+				)
+			)
+		)
+		(pin "6"
+		)
+		(pin "7"
+		)
+		(pin "8"
+		)
+		(pin "9"
+		)
+		(pin "10"
+		)
+		(pin "11"
+		)
+		(pin "12"
+		)
+		(pin "13"
+		)
+		(pin "14"
+		)
+		(pin "15"
+		)
+		(pin "16"
+		)
+		(pin "2"
+		)
+		(pin "3"
+		)
+		(pin "4"
+		)
+		(pin "5"
+		)
+		(pin "1"
+		)
+		(instances
+			(project "P.003-V1.0.1"
+				(path "/df58d102-266a-4360-93d3-4f9112ea1c17/0ae06492-67cd-4ae2-b1d8-141278a1bb86"
+					(reference "U2")
+					(unit 1)
+				)
+			)
+		)
+	)
 )

Commit message: Schematic wired
Connections:
- net VIN+: now also U2.10 (~{SRCLR}), U2.16 (VCC)
- net VIN-: now also U2.13 (~{OE}), U2.8 (GND)
- net Q1: now reaches U2.1 (QB)
- net CLK: now reaches U2.11 (SRCLK)
- net Latch: now reaches U2.12 (RCLK)
- net Data: now reaches U2.14 (SER)
- net Q0: now reaches U2.15 (QA)
- net Q2: now reaches U2.2 (QC)
- net Q3: now reaches U2.3 (QD)
- net Q4: now reaches U2.4 (QE)
- net Q5: now reaches U2.5 (QF)
- net Q6: now reaches U2.6 (QG)
- net Q7: now reaches U2.7 (QH)
- no-connect marks 0 -> 1
Other:
- company: (none) -> GSAS - Labs
- title: (none) -> Shift Register - 74HC595
- moved on the sheet: U2

Commit message: add footprint
Parts:
- U2: footprint (none) -> Package_DIP:DIP-16_W7.62mm
Changed lines of the file:
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@@
 			)
 		)
-		(property "Footprint" ""
+		(property "Footprint" "Package_DIP:DIP-16_W7.62mm"
 			(at 134.62 88.9 0)
 			(hide yes)
